File: pnid/schematics/lamarr/lamarr.kicad_sch (KiCad schematic)
At the start: 71 parts, among them U1 sound_supression:sensor

Commit message: dump of changes hotfire prep
Parts:
- ox_tanking_valve: renamed from tanking_valve?; value tanking_valve:sensor -> ox_tanking_valve:sensor
Connections:
- net at engine.~ (O): now also thrust.~; no longer ox_venturi.~
- net at fuel_venturi.~: now also CheckValve?.~, fuel_main_valve.~, fuel_venturi_pressure.~; no longer engine.~ (O)
- net at ox_pressure_regulator.~: now also ox_manual_valve?.~; no longer ox_needle_valve.~
- net at ox_manual_valve?.~: now also N2.~; no longer ox_pressure_regulator.~
- new net: fuel_manual_3way?.~, ox_pressurant_pressure:sensor.~, ox_pressurize_solenoid.~, ox_purge_solenoid.~
- new net: fuel_manual_3way.~, fuel_pressurant_pressure.~, fuel_pressurize_solenoid.~, fuel_purge_solenoid.~
- new net: Fuel.~, fuel_depressurize_solenoid.~, fuel_manual_vent_valve.~, fuel_pressurize_solenoid.~, fuel_safety_valve.~, fuel_tank_pressure.~
- new net: CheckValve?.~, LOX.~, ox_depressurize_solenoid.~, ox_manual_vent_valve.~, ox_safety_valve.~, ox_tank_pressure.~
- new net: LOX.~, ox_main_valve.~, ox_manual_tanking_valve.~
- new net: Fuel.~, fuel_main_valve.~, fuel_manual_tanking_valve.~
- new net: engine.~ (O), ox_venturi.~
- new net: engine.~ (O), fuel_venturi.~
- new net: Dewar.~, DewarOverPressureValve?.~, dewar_pressure?.~, dewar_pressurize_solenoid?.~
- new net: ox_needle_valve.~, ox_pressure_regulator.~
Changed lines of the file:
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@@
 		)
 		(property "Value" "ox_pressurize_solenoid:sensor"
-			(at 112.522 56.388 90)
+			(at 123.444 56.388 90)
 			(effects
 				(font
@@
 		)
 		(property "Value" "ox_purge_solenoid:sensor"
-			(at 122.174 109.982 90)
+			(at 116.332 109.982 90)
 			(effects
 				(font
@@
 		)
 		(property "Value" "fuel_purge_solenoid:sensor"
-			(at 80.772 110.236 90)
+			(at 86.868 109.982 90)
 			(effects
 				(font
 					(size 0.508 0.508)
 				)
-				(justify right)
+				(justify left)
 			)
 		)
@@
 		(on_board yes)
 		(dnp no)
-		(property "Reference" "tanking_valve?"
+		(property "Reference" "ox_tanking_valve"
 			(at 172.466 151.5618 0)
 			(effects
@@
 			)
 		)
-		(property "Value" "tanking_valve:sensor"
-			(at 172.466 150.114 0)
+		(property "Value" "ox_tanking_valve:sensor"
+			(at 172.466 170.688 0)
 			(effects
 				(font
@@
 			(project ""
 				(path "/604fc9f3-63a6-4133-afd1-4a5c2507dc1d"
-					(reference "tanking_valve?")
+					(reference "ox_tanking_valve")
 					(unit 1)
 				)
@@
 		)
 		(property "Value" "fuel_tank_pressure:sensor"
-			(at 69.85 80.518 0)
+			(at 80.518 71.374 0)
 			(effects
 				(font
@@
 		)
 		(property "Value" "ox_tank_pressure:sensor"
-			(at 122.428 80.264 0)
+			(at 122.936 71.374 0)
 			(effects
 				(font
@@
 		)
 		(property "Value" "ox_weight:sensor"
-			(at 126.238 146.812 0)
+			(at 123.698 145.542 0)
 			(effects
 				(font
@@
 		)
 		(property "Value" "tank_heating:sensor"
-			(at 123.698 113.792 0)
+			(at 123.698 111.252 0)
 			(effects
 				(font

Commit message: commit fixes/changes from electronics & software check
Parts:
- ox_purge_solenoid1: symbol PnID-Lib:Valve_Solenoid_NC -> PnID-Lib:Valve_Solenoid_NO
Connections:
- net at engine.~ (O): now also thrust.~; no longer ox_venturi.~
- net at fuel_venturi.~: now also CheckValve?.~, fuel_main_valve.~, fuel_venturi_pressure.~; no longer engine.~ (O)
- net at ox_pressure_regulator.~: now also ox_manual_valve?.~; no longer ox_needle_valve.~
- net at ox_manual_valve?.~: now also N2.~; no longer ox_pressure_regulator.~
- new net: fuel_manual_3way?.~, ox_pressurant_pressure:sensor.~, ox_pressurize_solenoid.~, ox_purge_solenoid.~
- new net: fuel_manual_3way.~, fuel_pressurant_pressure.~, fuel_pressurize_solenoid.~, fuel_purge_solenoid.~
- new net: Fuel.~, fuel_depressurize_solenoid.~, fuel_manual_vent_valve.~, fuel_pressurize_solenoid.~, fuel_safety_valve.~, fuel_tank_pressure.~
- new net: CheckValve?.~, LOX.~, ox_depressurize_solenoid.~, ox_manual_vent_valve.~, ox_safety_valve.~, ox_tank_pressure.~
- new net: LOX.~, ox_main_valve.~, ox_manual_tanking_valve.~
- new net: Fuel.~, fuel_main_valve.~, fuel_manual_tanking_valve.~
- new net: engine.~ (O), ox_venturi.~
- new net: engine.~ (O), fuel_venturi.~
- new net: Dewar.~, DewarOverPressureValve?.~, dewar_pressure?.~, dewar_pressurize_solenoid?.~
- new net: ox_needle_valve.~, ox_pressure_regulator.~
Changed lines of the file:
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@@
 	(wire
 		(pts
-			(xy 96.52 45.212) (xy 96.52 104.902)
+			(xy 98.552 45.212) (xy 98.552 104.902)
 		)
 		(stroke
@@
 	(wire
 		(pts
-			(xy 106.68 45.212) (xy 135.382 45.212)
+			(xy 104.648 45.212) (xy 135.382 45.212)
 		)
 		(stroke
@@
 	(wire
 		(pts
-			(xy 106.68 45.212) (xy 106.68 104.902)
+			(xy 104.648 45.212) (xy 104.648 104.902)
 		)
 		(stroke
@@
 	(wire
 		(pts
-			(xy 68.326 45.212) (xy 96.52 45.212)
+			(xy 68.326 45.212) (xy 98.552 45.212)
 		)
 		(stroke
@@
 	(wire
 		(pts
-			(xy 96.52 104.902) (xy 85.852 104.902)
+			(xy 98.552 104.902) (xy 85.852 104.902)
 		)
 		(stroke
@@
 	(wire
 		(pts
-			(xy 106.68 104.902) (xy 117.348 104.902)
+			(xy 104.648 104.902) (xy 117.348 104.902)
 		)
 		(stroke
@@
 		)
 		(property "Value" "fuel_pressurant_pressure:sensor"
-			(at 43.688 45.212 0)
+			(at 55.372 45.212 0)
 			(effects
 				(font
@@
 		)
 		(property "Value" "ox_pressurize_solenoid:sensor"
-			(at 123.444 56.388 90)
+			(at 124.714 56.388 90)
 			(effects
 				(font
@@
 		)
 		(property "Value" "fuel_pressurize_solenoid:sensor"
-			(at 80.01 56.388 90)
+			(at 78.994 56.388 90)
 			(effects
 				(font
@@
 		)
 		(property "Value" "ox_purge_solenoid:sensor"
-			(at 116.332 109.982 90)
+			(at 115.824 112.014 90)
 			(effects
 				(font
@@
 		)
 		(property "Value" "fuel_purge_solenoid:sensor"
-			(at 86.868 109.982 90)
+			(at 87.122 107.95 90)
 			(effects
 				(font
@@
 	)
 	(symbol
-		(lib_name "PnID-Lib:CheckValve")
 		(lib_id "PnID-Lib:CheckValve")
 		(at 135.382 66.548 270)
@@
 	)
 	(symbol
-		(lib_name "PnID-Lib:Tank_Slim")
 		(lib_id "PnID-Lib:Tank_Slim")
 		(at 135.382 129.794 0)
@@
 	)
 	(symbol
-		(lib_name "PnID-Lib:Tank_Slim")
 		(lib_id "PnID-Lib:Tank_Slim")
 		(at 68.326 129.794 0)
@@
 	)
 	(symbol
-		(lib_name "PnID-Lib:Engine")
 		(lib_id "PnID-Lib:Engine")
 		(at 101.854 182.626 0)
@@
 	)
 	(symbol
-		(lib_name "PnID-Lib:CheckValve")
 		(lib_id "PnID-Lib:CheckValve")
 		(at 85.852 131.064 270)
@@
 	)
 	(symbol
-		(lib_name "PnID-Lib:CheckValve")
 		(lib_id "PnID-Lib:CheckValve")
 		(at 117.348 131.064 270)
@@
 		)
 		(property "Value" "chamber_pressure:sensor"
-			(at 118.364 185.166 0)
+			(at 117.602 185.166 0)
 			(effects
 				(font
@@
 	)
 	(symbol
-		(lib_name "PnID-Lib:Valve_Manual")
 		(lib_id "PnID-Lib:Valve_Manual")
 		(at 147.066 162.814 0)
@@
 	)
 	(symbol
-		(lib_name "PnID-Lib:Venturi")
 		(lib_id "PnID-Lib:Venturi")
 		(at 109.22 171.45 270)
@@
 	)
 	(symbol
-		(lib_name "PnID-Lib:Venturi")
 		(lib_id "PnID-Lib:Venturi")
 		(at 94.488 171.45 270)
@@
 	)
 	(symbol
-		(lib_name "PnID-Lib:Valve_Manual")
 		(lib_id "PnID-Lib:Valve_Manual")
 		(at 25.908 41.656 90)
@@
 	)
 	(symbol
-		(lib_name "PnID-Lib:PressureRegulator")
 		(lib_id "PnID-Lib:PressureRegulator")
 		(at 36.576 30.988 0)
@@
 	)
 	(symbol
-		(lib_name "PnID-Lib:Valve_Needle")
 		(lib_id "PnID-Lib:Valve_Needle")
 		(at 52.578 30.988 0)
@@
 	)
 	(symbol
-		(lib_name "PnID-Lib:Valve_Manual_3Way")
 		(lib_id "PnID-Lib:Valve_Manual_3Way")
 		(at 68.326 38.1 0)
@@
 	)
 	(symbol
-		(lib_name "PnID-Lib:Valve_OverPressure")
 		(lib_id "PnID-Lib:Valve_OverPressure")
 		(at 41.656 83.82 0)
@@
 	)
 	(symbol
-		(lib_name "PnID-Lib:Valve_Solenoid_NO")
 		(lib_id "PnID-Lib:Valve_Solenoid_NO")
 		(at 54.864 71.374 0)
@@
 	)
 	(symbol
-		(lib_name "PnID-Lib:Valve_Manual")
 		(lib_id "PnID-Lib:Valve_Manual")
 		(at 57.15 162.814 0)
@@
 	)
 	(symbol
-		(lib_name "PnID-Lib:Valve_Manual")
 		(lib_id "PnID-Lib:Valve_Manual")
 		(at 41.402 98.044 0)
@@
 	)
 	(symbol
-		(lib_name "PnID-Lib:Valve_Servo")
 		(lib_id "PnID-Lib:Valve_Servo")
 		(at 79.502 162.814 0)
@@
 	)
 	(symbol
-		(lib_name "PnID-Lib:Valve_Solenoid_NC")
 		(lib_id "PnID-Lib:Valve_Solenoid_NC")
 		(at 230.378 129.54 0)
@@
 	)
 	(symbol
-		(lib_name "PnID-Lib:Valve_OverPressure")
 		(lib_id "PnID-Lib:Valve_OverPressure")
 		(at 216.154 143.51 90)
@@
 	)
 	(symbol
-		(lib_name "PnID-Lib:Tank_Slim")
 		(lib_id "PnID-Lib:Tank_Slim")
 		(at 188.976 147.066 0)
@@
 	)
 	(symbol
-		(lib_name "PnID-Lib:Valve_Servo")
 		(lib_id "PnID-Lib:Valve_Servo")
 		(at 172.466 162.814 0)
@@
 	)
 	(symbol
-		(lib_name "PnID-Lib:Valve_OverPressure")
 		(lib_id "PnID-Lib:Valve_OverPressure")
 		(at 162.052 83.82 0)
@@
 	)
 	(symbol
-		(lib_name "PnID-Lib:Valve_Solenoid_NO")
 		(lib_id "PnID-Lib:Valve_Solenoid_NO")
 		(at 148.844 71.374 0)
@@
 	)
 	(symbol
-		(lib_name "PnID-Lib:Valve_Manual")
 		(lib_id "PnID-Lib:Valve_Manual")
 		(at 162.306 98.044 0)
@@
 		)
 		(property "Value" "fuel_tank_pressure:sensor"
-			(at 80.518 71.374 0)
+			(at 80.01 71.374 0)
 			(effects
 				(font
@@
 		)
 		(property "Value" "ox_tank_pressure:sensor"
-			(at 122.936 71.374 0)
+			(at 123.444 71.374 0)
 			(effects
 				(font
@@
 	)
 	(symbol
-		(lib_name "PnID-Lib:PressureRegulator")
 		(lib_id "PnID-Lib:PressureRegulator")
 		(at 167.132 30.988 0)
@@
 	)
 	(symbol
-		(lib_name "PnID-Lib:Valve_Needle")
 		(lib_id "PnID-Lib:Valve_Needle")
 		(at 151.13 30.988 0)
@@
 	)
 	(symbol
-		(lib_name "PnID-Lib:Valve_Manual_3Way")
 		(lib_id "PnID-Lib:Valve_Manual_3Way")
 		(at 135.382 38.1 0)
@@
 	)
 	(symbol
-		(lib_name "PnID-Lib:Valve_Servo")
 		(lib_id "PnID-Lib:Valve_Servo")
 		(at 123.698 162.814 0)
@@
 		)
 		(property "Value" "thrust:sensor"
-			(at 78.232 185.166 0)
+			(at 86.36 185.166 0)
 			(effects
 				(font
 					(size 0.508 0.508)
 				)
-				(justify right)
+				(justify left)
 			)
 		)
@@
 	)
 	(symbol
-		(lib_name "PnID-Lib:Valve_Manual")
 		(lib_id "PnID-Lib:Valve_Manual")
 		(at 177.8 41.656 270)
@@
 	)
 	(symbol
-		(lib_name "PnID-Lib:Valve_Needle")
 		(lib_id "PnID-Lib:Valve_Needle")
 		(at 247.142 129.54 0)
@@
 	)
 	(symbol
-		(lib_name "PnID-Lib:PressureRegulator")
 		(lib_id "PnID-Lib:PressureRegulator")
 		(at 263.144 129.54 0)
@@
 	)
 	(symbol
-		(lib_name "PnID-Lib:Valve_Manual")
 		(lib_id "PnID-Lib:Valve_Manual")
 		(at 273.812 140.208 270)
@@
 		)
 		(property "Value" "fuel_weight:sensor"
-			(at 43.942 139.954 0)
+			(at 49.276 139.954 0)
 			(effects
 				(font
 					(size 0.508 0.508)
 				)
+				(justify left)
 			)
 		)
@@
 		)
 		(property "Value" "ox_weight:sensor"
-			(at 123.698 145.542 0)
+			(at 125.222 145.542 0)
 			(effects
 				(font
@@
 		)
 		(property "Value" "tank_heating:sensor"
-			(at 123.698 111.252 0)
+			(at 124.968 111.76 0)
 			(effects
 				(font
@@
 	)
 	(symbol
-		(lib_name "PnID-Lib:Valve_Solenoid_NC")
-		(lib_id "PnID-Lib:Valve_Solenoid_NC")
+		(lib_name "Valve_Solenoid_NO_1")
+		(lib_id "PnID-Lib:Valve_Solenoid_NO")
 		(at 57.404 174.752 90)
 		(unit 1)
@@
 		)
 		(property "Value" "safety_valves:sensor"
-			(at 44.704 174.752 90)
+			(at 45.974 175.006 90)
 			(effects
 				(font
@@
 		)
 		(property "Value" "sound_supression:sensor"
-			(at 45.4664 186.7301 0)
+			(at 45.72 186.69 0)
 			(effects
 				(font

Commit message: commit before hotfire
Parts:
- removed heater1: tank_heating:sensor, symbol PnID-Lib:heater
- removed ox_weight: ox_weight:sensor, symbol PnID-Lib:Sensor_Load_Short
- added ox_weight: ox_weight:sensor, symbol PnID-Lib:Sensor_Load
- safety_valves: renamed from ox_purge_solenoid1; symbol PnID-Lib:Valve_Solenoid_NO -> PnID-Lib:Valve_Solenoid_NC
Connections:
- net at engine.~ (O): now also thrust.~; no longer ox_venturi.~
- net at fuel_venturi.~: now also CheckValve?.~, fuel_main_valve.~, fuel_venturi_pressure.~; no longer engine.~ (O)
- net at ox_pressure_regulator.~: now also ox_manual_valve?.~; no longer ox_needle_valve.~
- net at ox_manual_valve?.~: now also N2.~; no longer ox_pressure_regulator.~
- new net: fuel_manual_3way?.~, ox_pressurant_pressure:sensor.~, ox_pressurize_solenoid.~, ox_purge_solenoid.~
- new net: fuel_manual_3way.~, fuel_pressurant_pressure.~, fuel_pressurize_solenoid.~, fuel_purge_solenoid.~
- new net: Fuel.~, fuel_depressurize_solenoid.~, fuel_manual_vent_valve.~, fuel_pressurize_solenoid.~, fuel_safety_valve.~, fuel_tank_pressure.~
- new net: CheckValve?.~, LOX.~, ox_depressurize_solenoid.~, ox_manual_vent_valve.~, ox_safety_valve.~, ox_tank_pressure.~
- new net: LOX.~, ox_main_valve.~, ox_manual_tanking_valve.~
- new net: Fuel.~, fuel_main_valve.~, fuel_manual_tanking_valve.~
- new net: engine.~ (O), ox_venturi.~
- new net: engine.~ (O), fuel_venturi.~
- new net: Dewar.~, DewarOverPressureValve?.~, dewar_pressure?.~, dewar_pressurize_solenoid?.~
- new net: ox_needle_valve.~, ox_pressure_regulator.~
