File: pnid/schematics/lamarr/propulsion_teststand.kicad_sch (KiCad schematic)
At the start: 18 parts

Commit message: improve label placement for remaining pnids
Connections:
- new net: Valve_Manual_3Way.~, pressurantPressureRegulator.~, pressurant_pressure.~, pressurant_tank.~
- new net: CheckValve?.~, Tank.~, tank_pressure.~
- now unconnected: pressurant_tank.~
Changed lines of the file:
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@@
 		)
 		(property "Value" "pressurant_pressure:sensor"
-			(at 151.13 60.198 0)
+			(at 145.796 60.198 0)
 			(effects
 				(font
@@
 	)
 	(symbol
-		(lib_name "PnID-Lib:CheckValve")
 		(lib_id "PnID-Lib:CheckValve")
 		(at 133.35 102.108 270)
@@
 	)
 	(symbol
-		(lib_name "PnID-Lib:Tank_Slim")
 		(lib_id "PnID-Lib:Tank_Slim")
 		(at 133.35 128.27 0)
@@
 		)
 		(property "Value" "venturi_pressure:sensor"
-			(at 109.982 159.766 0)
-			(effects
-				(font
-					(size 0.508 0.508)
-				)
+			(at 119.126 159.766 0)
+			(effects
+				(font
+					(size 0.508 0.508)
+				)
+				(justify left)
 			)
 		)
@@
 	)
 	(symbol
-		(lib_name "PnID-Lib:Venturi")
 		(lib_id "PnID-Lib:Venturi")
 		(at 133.35 168.656 270)
@@
 		)
 		(property "Value" "venturi:sensor"
-			(at 138.176 168.656 90)
+			(at 139.446 168.656 90)
 			(effects
 				(font
@@
 	)
 	(symbol
-		(lib_name "PnID-Lib:Valve_Manual")
 		(lib_id "PnID-Lib:Valve_Manual")
 		(at 76.708 58.928 90)
@@
 	)
 	(symbol
-		(lib_name "PnID-Lib:PressureRegulator")
 		(lib_id "PnID-Lib:PressureRegulator")
 		(at 86.36 48.26 0)
@@
 		)
 		(property "Value" "tank_pressure:sensor"
-			(at 114.3 106.934 0)
+			(at 119.126 106.934 0)
 			(effects
 				(font
@@
 		)
 		(property "Value" "main_valve:sensor"
-			(at 109.982 151.13 90)
-			(effects
-				(font
-					(size 0.508 0.508)
-				)
+			(at 119.126 151.13 90)
+			(effects
+				(font
+					(size 0.508 0.508)
+				)
+				(justify left)
 			)
 		)
@@
 	)
 	(symbol
-		(lib_name "PnID-Lib:Tank_Slim")
 		(lib_id "PnID-Lib:Tank_Slim")
 		(at 133.35 45.212 0)
@@
 	)
 	(symbol
-		(lib_name "PnID-Lib:Valve_Manual")
 		(lib_id "PnID-Lib:Valve_Manual")
 		(at 100.838 48.26 0)
@@
 	)
 	(symbol
-		(lib_name "propulsion_teststand-rescue:Valve_Manual_3Way-PnID-Lib")
 		(lib_id "propulsion_teststand-rescue:Valve_Manual_3Way-PnID-Lib")
 		(at 117.348 60.198 90)
@@
 		)
 		(property "Value" "pressurant_valve:sensor"
-			(at 109.474 89.662 90)
-			(effects
-				(font
-					(size 0.508 0.508)
-				)
+			(at 119.126 89.662 90)
+			(effects
+				(font
+					(size 0.508 0.508)
+				)
+				(justify left)
 			)
 		)
@@
 	)
 	(symbol
-		(lib_name "PnID-Lib:PressureRegulator")
 		(lib_id "PnID-Lib:PressureRegulator")
 		(at 133.35 75.692 90)
@@
 		)
 		(property "Value" "venturi_weight:sensor"
-			(at 109.728 168.656 0)
-			(effects
-				(font
-					(size 0.508 0.508)
-				)
-			)
-		)
+			(at 119.126 168.656 0)
+			(effects
+				(font
+					(size 0.508 0.508)
+				)
+				(justify left)
+			)
+		)

Commit message: pre-branch merge commit
Parts:
- fuel_main_valve: renamed from main_valve; value main_valve:sensor -> fuel_main_valve:sensor
- fuel_pressurant_valve: renamed from pressurant_valve; value pressurant_valve:sensor -> fuel_pressurant_valve:sensor
- fuel_weight: renamed from venturi_weight; value venturi_weight:sensor -> fuel_weight:sensor
- pressurant_pressure: value pressurant_pressure:sensor -> fuel_rocket_pressurant_pressure:sensor
- tank_pressure: value tank_pressure:sensor -> fuel_rocket_tank_pressure:sensor
- venturi_pressure: value venturi_pressure:sensor -> fuel_venturi_pressure:sensor
Connections:
- new net: Valve_Manual_3Way.~, pressurantPressureRegulator.~, pressurant_pressure.~, pressurant_tank.~
- new net: CheckValve?.~, Tank.~, tank_pressure.~
- now unconnected: pressurant_tank.~
Changed lines of the file:
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@@
 			)
 		)
-		(property "Value" "pressurant_pressure:sensor"
+		(property "Value" "fuel_rocket_pressurant_pressure:sensor"
 			(at 145.796 60.198 0)
 			(effects
@@
 			)
 		)
-		(property "Value" "venturi_pressure:sensor"
+		(property "Value" "fuel_venturi_pressure:sensor"
 			(at 119.126 159.766 0)
 			(effects
@@
 			)
 		)
-		(property "Value" "tank_pressure:sensor"
+		(property "Value" "fuel_rocket_tank_pressure:sensor"
 			(at 119.126 106.934 0)
 			(effects
@@
 		(on_board yes)
 		(dnp no)
-		(property "Reference" "main_valve"
+		(property "Reference" "fuel_main_valve"
 			(at 122.0978 151.13 0)
 			(effects
@@
 			)
 		)
-		(property "Value" "main_valve:sensor"
+		(property "Value" "fuel_main_valve:sensor"
 			(at 119.126 151.13 90)
 			(effects
@@
 			(project "propulsion_teststand"
 				(path "/92b2e49c-6691-4975-bb0e-16f530c919c8"
-					(reference "main_valve")
+					(reference "fuel_main_valve")
 					(unit 1)
 				)
@@
 		(on_board yes)
 		(dnp no)
-		(property "Reference" "pressurant_valve"
+		(property "Reference" "fuel_pressurant_valve"
 			(at 137.8712 89.1032 90)
 			(effects
@@
 			)
 		)
-		(property "Value" "pressurant_valve:sensor"
+		(property "Value" "fuel_pressurant_valve:sensor"
 			(at 119.126 89.662 90)
 			(effects
@@
 			(project "propulsion_teststand"
 				(path "/92b2e49c-6691-4975-bb0e-16f530c919c8"
-					(reference "pressurant_valve")
+					(reference "fuel_pressurant_valve")
 					(unit 1)
 				)
@@
 		(on_board yes)
 		(dnp no)
-		(property "Reference" "venturi_weight"
+		(property "Reference" "fuel_weight"
 			(at 125.9332 161.4678 0)
 			(effects
@@
 			)
 		)
-		(property "Value" "venturi_weight:sensor"
+		(property "Value" "fuel_weight:sensor"
 			(at 119.126 168.656 0)
 			(effects
@@
 			(project "propulsion_teststand"
 				(path "/92b2e49c-6691-4975-bb0e-16f530c919c8"
-					(reference "venturi_weight")
-					(unit 1)
-				)
+					(reference "fuel_weight")
+					(unit 1)
+				)
