File: pnid/schematics/lamarr/lamarr_half_static.kicad_sch (KiCad schematic)
At the start: 65 parts, among them U1 sound_supression:sensor

Commit message: Mapping for Rocket
Connections:
- net at engine.~ (O): now also venturi1.~; no longer ox_venturi.~
- net at venturi1.~: now also fuel_main_valve1.~, venturi_pressure1.~; no longer engine.~ (O)
- net at ox_pressure_regulator.~: now also ox_manual_valve?.~; no longer ox_needle_valve.~
- net at ox_manual_valve?.~: now also N2.~; no longer ox_pressure_regulator.~
- net at fuel_safety_valve.~: now also fuel_main_valve1.~; no longer Tank1.~
- new net: fuel_manual_3way?.~, ox_pressurant_pressure:sensor.~, ox_pressurize_solenoid.~, ox_purge_solenoid.~
- new net: CheckValve?.~, LOX.~, ox_depressurize_solenoid.~, ox_manual_vent_valve.~, ox_safety_valve.~, ox_tank_pressure.~
- new net: engine.~ (O), ox_venturi.~
- new net: Dewar.~, DewarOverPressureValve?.~, dewar_pressure?.~, dewar_pressurize_solenoid?.~
- new net: ox_needle_valve.~, ox_pressure_regulator.~
- new net: Tank1.~, fuel_safety_valve.~
- new net: Valve_Manual_3Way1.~, pressurantPressureRegulator1.~, pressurant_pressure1.~, pressurant_tank1.~
- now unconnected: pressurant_tank1.~
Changed lines of the file:
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@@
 	)
 	(symbol
-		(lib_name "PnID-Lib:Valve_Solenoid_NC")
 		(lib_id "PnID-Lib:Valve_Solenoid_NC")
 		(at 109.22 93.98 90)
@@
 	)
 	(symbol
-		(lib_name "PnID-Lib:Tank_Slim")
 		(lib_id "PnID-Lib:Tank_Slim")
 		(at 135.382 117.094 0)
@@
 	)
 	(symbol
-		(lib_name "PnID-Lib:CheckValve")
 		(lib_id "PnID-Lib:CheckValve")
 		(at 109.22 113.284 270)
@@
 	)
 	(symbol
-		(lib_name "PnID-Lib:Tank_Slim")
 		(lib_id "PnID-Lib:Tank_Slim")
 		(at 82.804 116.586 0)
@@
 	)
 	(symbol
-		(lib_name "PnID-Lib:Venturi")
 		(lib_id "PnID-Lib:Venturi")
 		(at 83.058 171.45 270)
@@
 	)
 	(symbol
-		(lib_name "PnID-Lib:Valve_Servo")
 		(lib_id "PnID-Lib:Valve_Servo")
 		(at 83.058 155.956 90)
