File: pnid/schematics/lamarr/lamarr_gn.kicad_sch (KiCad schematic)
At the start: 16 parts

Commit message: various fixes
configure lora use,
fix guidance & navigation pnid,
fix retract threshold
Parts:
- removed ecu_flash_status: ecu:FlashStatus, symbol PnID-Lib:LED
- removed rcu_flash_status: rcu:FlashStatus, symbol PnID-Lib:LED
- added Engine: engine_ecu:FlashStatus, symbol PnID-Lib:LED
- added Fuel: fuel_ecu:FlashStatus, symbol PnID-Lib:LED
- added Fuel: fuel_ecu:LoggingEnabled, symbol PnID-Lib:LED
- added Ox: ox_ecu:LoggingEnabled, symbol PnID-Lib:LED
- added Ox: ox_ecu:FlashStatus, symbol PnID-Lib:LED
- added RCU: rcu:FlashStatus, symbol PnID-Lib:LED
- Engine: renamed from ecu_logging_en; value ecu:LoggingEnabled -> engine_ecu:LoggingEnabled
- renumbered rcu_logging_en to RCU

Commit message: i mog schlafn
Parts:
- Accel_X: value accel_x -> rcu_accel_x:sensor
- Accel_Y: value accel_y -> rcu_accel_y:sensor
- Accel_Z: value accel_z -> rcu_accel_z:sensor
Changed lines of the file:
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@@
 			)
 		)
-		(property "Value" "accel_y"
+		(property "Value" "rcu_accel_y:sensor"
 			(at 63.754 134.366 0)
 			(effects
@@
 			)
 		)
-		(property "Value" "accel_z"
+		(property "Value" "rcu_accel_z:sensor"
 			(at 34.798 159.766 0)
 			(effects
@@
 			)
 		)
-		(property "Value" "accel_x"
+		(property "Value" "rcu_accel_x:sensor"
 			(at 34.798 134.366 0)
 			(effects
