File: pnid/schematics/lamarr/lamarr_hedy_vertical.kicad_sch (KiCad schematic)
At the start: 103 parts, among them U1 Rocket_Big, U2 ox_sense_12V:sensor

Commit message: more refinements in sensor calibration & ECUI look
Parts:
- removed ox_decoupler_temperature: engine_temp_1:sensor, symbol PnID-Lib:Sensor_Temperature
- removed ox_decoupler_temperature1: ox_temp_0:sensor, symbol PnID-Lib:Sensor_Temperature
- added fuel_main_valve_servo_temperature: engine_temp_1:sensor, symbol PnID-Lib:Sensor_Temperature
- added ox_vent_temperature: ox_temp_0:sensor, symbol PnID-Lib:Sensor_Temperature
- Retract: renamed from Motor1; symbol PnID-Lib:Motor -> PnID-Lib:Retract
- engine_ECU_temperature: value engine_temp_0:sensor -> fuel_temp_1:sensor
- igniter1: value internal_igniter_1_cont:sensor -> internal_igniter_1:sensor
- igniter2: value internal_igniter_2_cont:sensor -> internal_igniter_2:sensor
- ox_main_valve_servo_temperature: value fuel_temp_1:sensor -> engine_temp_0:sensor
- voltmeter1: value internal_igniter_1:sensor -> internal_igniter_1_cont:sensor; symbol PnID-Lib:voltmeter -> PnID-Lib:continuity
- voltmeter2: value internal_igniter_2:sensor -> internal_igniter_2_cont:sensor; symbol PnID-Lib:voltmeter -> PnID-Lib:continuity
Connections:
- net at engine.~ (C): now also venturi1.~
- net at ox_venturi.~: now also ox_main_valve.~, ox_venturi_pressure.~; no longer engine.~ (C)
- net at venturi1.~: now also fuel_main_valve.~, fuel_venturi_pressure.~; no longer engine.~ (C)
- net at dewar_needle_valve?.~: now also C2.~, C3.~, press_in.~; no longer C1.~
- new net: engine.~ (C), ox_venturi.~
- new net: OX.~, ox_main_valve.~, ox_quick_connect.~
- new net: DewarOverPressureValve?.~, LOX.~, dewar_pressurize_solenoid.~
- new net: C1.~, dewar_needle_valve?.~
- new net: ox_pressurant_valve.~, ox_pressurant_vent_valve.~, pressurantPressureRegulator2.~
- new net: FUEL.~, fuel_main_valve.~, ox_quick_connect1.~
- new net: fuel_pressurant_valve.~, fuel_pressurant_vent_valve.~, pressurantPressureRegulator1.~
